File: wrover_the_thesis.kicad_pcb (KiCad board)
At the start: 2 copper layers, 40.9 x 63.5 mm, 44 parts, among them J4 CAN_out, J5 Conn_02x03_Counter_Clockwise, J6 Conn_02x03_Counter_Clockwise, J7 Conn_02x03_Counter_Clockwise, Q3 Q_NPN_BCE, Q4 Q_NPN_BCE, SW1 reset, SW2 boot, U1 ESP32-WROVER-B_(16MB), U2 CP2102N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

Commit message: update
Parts:
- removed J6, J7: Conn_02x03_Counter_Clockwise, Connector_PinHeader_2.54mm:PinHeader_2x03_P2.54mm_Vertical
- removed Power: Barrel_Jack_Switch, Connector_BarrelJack:BarrelJack_Wuerth_6941xx301002
- added J3: Barrel_Jack_Switch, Connector_BarrelJack:BarrelJack_Wuerth_6941xx301002, F.Cu at (86.2, 91.4)
- added J9: USB_B_Micro, Connector_USB:USB_Micro-B_Wuerth_629105150521, F.Cu at (76.1, 99.1)
- added R23: 1K, Resistor_SMD:R_0603_1608Metric_Pad1.05x0.95mm_HandSolder, B.Cu at (67.4, 92.4)
- added R25: 10K, Resistor_SMD:R_0603_1608Metric_Pad1.05x0.95mm_HandSolder, B.Cu at (67.4, 88.7)
- added R26: 470, Resistor_SMD:R_0603_1608Metric_Pad1.05x0.95mm_HandSolder, B.Cu at (76.1, 88.6)
- added R27: 470, Resistor_SMD:R_0603_1608Metric_Pad1.05x0.95mm_HandSolder, B.Cu at (77.6, 88.6)
- added U7: CP2102N, Package_DFN_QFN:QFN-28-1EP_5x5mm_P0.5mm_EP3.35x3.35mm, B.Cu at (71.3, 90.6)
- moved J4 5.93 mm to (58.6, 77.8)
- moved C11 5.90 mm to (80.4, 94.1)
- moved J1 5.90 mm to (90.0, 79.9)
- moved J8 5.90 mm to (90.7, 69.5)
- moved Q3 5.90 mm to (65.8, 76.8)
- moved R12 5.90 mm to (73.2, 72.1)
- moved R14 5.90 mm to (80.2, 81.2)
- moved R16 5.90 mm to (69.3, 80.8)
- moved R4 5.90 mm to (73.5, 68.7)
- moved SW1 5.90 mm to (65.4, 90.7)
- moved R1 5.90 mm to (63.9, 84.9)
- moved C3 5.90 mm to (82.7, 89.5)
- moved C4 5.90 mm to (80.3, 88.8)
- moved D5 5.90 mm to (80.8, 77.2)
- moved R11 5.90 mm to (73.2, 73.6)
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- renumbered Flash to J1, COnn to J2, CAN_USB to J8, AMS to U3, CAN to U4
Routing:
- net HSPI_MISO: track 21.2 -> 56.1 mm
- net HSPI_MOSI: track 22.2 -> 55.3 mm
- net +5V: track 120.6 -> 145.3 mm
- net +3V3: track 200.5 -> 191.6 mm, vias 16 -> 17
- net Net-(J9-Pad3): track 0.00 -> 7.62 mm, vias 0 -> 1
- net Net-(J9-Pad2): track 0.00 -> 7.20 mm, vias 0 -> 1
- net Net-(R27-Pad2): track 0.00 -> 4.83 mm
- net Net-(R26-Pad2): track 0.00 -> 3.11 mm
- net Net-(R25-Pad1): track 0.00 -> 1.86 mm
- net Net-(R23-Pad2): track 0.00 -> 1.45 mm
- net GND: track 0.00 -> 0.71 mm, vias 280 -> 268
- net Net-(J10-Pad8): vias 0 -> 1
- net Net-(D7-Pad2): vias 0 -> 2
