File: wrover_the_thesis.sch (KiCad schematic (older format))
At the start: 44 parts, among them J1 USB_B_Micro, J2 Conn_02x13_Counter_Clockwise, J3 Barrel_Jack_Switch, J4 CAN_out, J5 Conn_02x03_Counter_Clockwise, J6 Conn_02x03_Counter_Clockwise, J7 Conn_02x03_Counter_Clockwise, J8 USB_C_Receptacle_USB2.0, Q3 Q_NPN_BCE, Q4 Q_NPN_BCE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

Commit message: update
Parts:
- removed J6, J7: Conn_02x03_Counter_Clockwise, Connector_PinHeader_2.54mm:PinHeader_2x03_P2.54mm_Vertical, symbol Connector_Generic:Conn_02x03_Counter_Clockwise
Other:
- note added: "pinout"
- note added: "power 12v\n"
- note added: "power 5V\n"
- moved on the sheet: C10, C11, C8, C9, J2, J3, J5, J8, U5
