File: esp_wrover_open.kicad_pcb (KiCad board)
At the start: 2 copper layers, 40.9 x 63.5 mm, 44 parts, among them J4 CAN_out, J5 Conn_02x03_Counter_Clockwise, J6 Conn_02x03_Counter_Clockwise, J7 Conn_02x03_Counter_Clockwise, Q3 Q_NPN_BCE, Q4 Q_NPN_BCE, SW1 reset, SW2 boot, U1 ESP32-WROVER-B_(16MB), U2 CP2102N, U5 LM1084-5.0

Commit message: update
Routing:
- net Net-(J1-Pad3): track 22.2 -> 17.0 mm, vias 0 -> 2
- net GND: vias 280 -> 277
Changed lines of the file:
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@@
     (thickness 1.6)
     (drawings 41)
-    (tracks 841)
+    (tracks 842)
     (zones 0)
     (modules 44)
@@
     (40 Dwgs.User user hide)
     (41 Cmts.User user)
-    (42 Eco1.User user)
+    (42 Eco1.User user hide)
     (43 Eco2.User user)
     (44 Edge.Cuts user)
     (45 Margin user)
-    (46 B.CrtYd user hide)
-    (47 F.CrtYd user)
+    (46 B.CrtYd user)
+    (47 F.CrtYd user hide)
     (48 B.Fab user)
     (49 F.Fab user hide)
@@
       (drillshape 0)
       (scaleselection 1)
-      (outputdirectory "Gerber/"))
+      (outputdirectory "gerber/"))
   )
   (net 0 "")
@@
   (via (at 63.95 60.58) (size 0.4) (drill 0.3) (layers F.Cu B.Cu) (net 1))
   (via (at 63.55 60.97) (size 0.4) (drill 0.3) (layers F.Cu B.Cu) (net 1))
-  (via (at 78.69 88.18) (size 0.8) (drill 0.4) (layers F.Cu B.Cu) (net 1))
-  (via (at 79.88 88.19) (size 0.8) (drill 0.4) (layers F.Cu B.Cu) (net 1))
-  (via (at 81.04 88.19) (size 0.8) (drill 0.4) (layers F.Cu B.Cu) (net 1))
   (via (at 61.23 78.67) (size 0.8) (drill 0.4) (layers F.Cu B.Cu) (net 1))
   (via (at 68.75 48.89) (size 0.8) (drill 0.4) (layers F.Cu B.Cu) (net 1))
@@
   (segment (start 60.55501 77.78499) (end 60.55501 75.93) (width 0.5) (layer F.Cu) (net 5))
   (segment (start 52.44 80.07) (end 58.27 80.07) (width 0.5) (layer F.Cu) (net 5))
-  (segment (start 86.44 85.245) (end 85.54 85.245) (width 0.25) (layer F.Cu) (net 6))
-  (segment (start 87.365001 86.170001) (end 86.44 85.245) (width 0.25) (layer F.Cu) (net 6))
-  (segment (start 87.365001 88.954937) (end 87.365001 86.170001) (width 0.25) (layer F.Cu) (net 6))
-  (segment (start 86.299928 90.02001) (end 87.365001 88.954937) (width 0.25) (layer F.Cu) (net 6))
-  (segment (start 74.005578 90.02001) (end 86.299928 90.02001) (width 0.25) (layer F.Cu) (net 6))
+  (segment (start 72.65 87.14) (end 72.65 88.664432) (width 0.25) (layer F.Cu) (net 6))
   (segment (start 72.65 88.664432) (end 74.005578 90.02001) (width 0.25) (layer F.Cu) (net 6))
-  (segment (start 72.65 87.14) (end 72.65 88.664432) (width 0.25) (layer F.Cu) (net 6))
+  (segment (start 74.005578 90.02001) (end 76.78999 90.02001) (width 0.25) (layer F.Cu) (net 6))
+  (via (at 76.78999 90.02001) (size 0.8) (drill 0.4) (layers F.Cu B.Cu) (net 6))
+  (segment (start 84.47174 85.245) (end 81.36674 88.35) (width 0.25) (layer F.Cu) (net 6))
+  (segment (start 85.54 85.245) (end 84.47174 85.245) (width 0.25) (layer F.Cu) (net 6))
+  (segment (start 81.36674 88.35) (end 79.26 88.35) (width 0.25) (layer F.Cu) (net 6))
+  (segment (start 79.26 88.35) (end 79.26 88.35) (width 0.25) (layer F.Cu) (net 6))
+  (via (at 79.26 88.35) (size 0.8) (drill 0.4) (layers F.Cu B.Cu) (net 6))
+  (segment (start 78.46 88.35) (end 79.26 88.35) (width 0.25) (layer B.Cu) (net 6))
+  (segment (start 76.78999 90.02001) (end 78.46 88.35) (width 0.25) (layer B.Cu) (net 6))
   (segment (start 84.64 85.895) (end 85.54 85.895) (width 0.25) (layer F.Cu) (net 7))
   (segment (start 81.43999 89.09501) (end 84.64 85.895) (width 0.25) (layer F.Cu) (net 7))

Commit message: cpmonent
Parts:
- removed C10, C8: 10uF, Resistor_SMD:R_1210_3225Metric
- removed C11, C9: 100nF, Capacitor_SMD:C_0603_1608Metric
- removed CAN: SN65HVD230, Package_SO:SOIC-8_3.9x4.9mm_P1.27mm
- removed COnn: Conn_02x13_Counter_Clockwise, Connector_PinHeader_2.54mm:PinHeader_2x13_P2.54mm_Vertical
- removed Flash: USB_B_Micro, Connector_USB:USB_Micro-B_Wuerth_629105150521
- removed J6, J7: Conn_02x03_Counter_Clockwise, Connector_PinHeader_2.54mm:PinHeader_2x03_P2.54mm_Vertical
- removed R14: 1K, Resistor_SMD:R_0603_1608Metric_Pad1.05x0.95mm_HandSolder
- removed the R3 at (67.9, 70.3)
- removed the R4 at (71.0, 74.1)
- removed the U2 at (72.7, 84.7)
- removed U5: LM1084-5.0, Package_TO_SOT_THT:TO-220-3_Vertical
- added J3: Conn_02x03_Counter_Clockwise, Connector_PinHeader_2.54mm:PinHeader_2x03_P2.54mm_Vertical, F.Cu at (70.0, 94.1)
- added U1: CP2104, Package_DFN_QFN:QFN-24-1EP_4x4mm_P0.5mm_EP2.6x2.6mm, F.Cu at (74.6, 78.6)
- J4: value CAN_out -> Conn_02x03_Counter_Clockwise; footprint Connector:JWT_A3963_1x02_P3.96mm_Vertical -> Connector_PinHeader_2.54mm:PinHeader_2x03_P2.54mm_Vertical
- J5: value Conn_02x03_Counter_Clockwise -> Conn_02x20_Counter_Clockwise; footprint Connector_PinHeader_2.54mm:PinHeader_2x03_P2.54mm_Vertical -> Connector_PinHeader_2.54mm:PinHeader_2x20_P2.54mm_Vertical
- moved SW2 50.8 mm to (88.4, 56.7)
- moved C2 50.8 mm to (86.8, 50.9)
- moved R2 50.8 mm to (90.0, 50.9)
- moved R1 37.1 mm to (87.0, 63.4)
- moved SW1 37.1 mm to (88.5, 69.2)
- moved C1 37.1 mm to (90.2, 63.4)
- moved J5 36.9 mm to (54.4, 45.9), turned to 0 degrees
- moved C5 20.9 mm to (65.4, 74.0), turned to 0 degrees
- moved U3 18.2 mm to (64.6, 79.2), turned to 90 degrees
- moved C3 16.3 mm to (66.0, 86.8), turned to 180 degrees
- moved C4 14.6 mm to (66.7, 84.5), turned to 180 degrees
- moved Q2 14.4 mm to (77.7, 86.8), turned to 270 degrees
- moved J4 12.2 mm to (61.2, 94.1), turned to 90 degrees
- moved Q1 11.4 mm to (73.8, 86.7), turned to 270 degrees
- moved R10 11.3 mm to (77.7, 83.2), turned to 0 degrees
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- renumbered D3 to D1, D4 to D2, D5 to D3, CAN_USB to J1, Power to J2, Q3 to Q1, Q4 to Q2, R16 to R10, R9 to R3, R10 to R4, R13 to R5, R15 to R6, R11 to R7, R12 to R8, R17 to R9, U1 to U2, AMS to U3
Connections:
- J1 pad A4: +12V -> +5V
- J1 pad A5: (no net) -> Net-(J1-PadA5)
- J1 pad A6: CAN_H -> Net-(J1-PadA6)
- J1 pad A7: CAN_L -> Net-(J1-PadA7)
- J1 pad A8: (no net) -> Net-(J1-PadA8)
- J1 pad A9: +12V -> +5V
- J1 pad B4: +12V -> +5V
- J1 pad B5: (no net) -> Net-(J1-PadB5)
- J1 pad B6: CAN_H -> Net-(J1-PadA6)
- J1 pad B7: CAN_L -> Net-(J1-PadA7)
- J1 pad B8: (no net) -> Net-(J1-PadB8)
- J1 pad B9: +12V -> +5V
- J4 pad 1: CAN_H -> +3V3
- J4 pad 2: CAN_L -> GND
- J5 pad 1: +12V -> EN
- J5 pad 2: GND -> RX0
- J5 pad 3: +12V -> TX0
- J5 pad 4: GND -> +5V
- J5 pad 5: +12V -> +3V3
- R7 pad 1: TX0 -> RX0
- R8 pad 1: RX0 -> TX0
- U2 pad 10: DAC1 -> Net-(U2-Pad10)
- U2 pad 11: DAC2 -> Net-(U2-Pad11)
- U2 pad 12: HSPI_SE -> Net-(U2-Pad12)
- U2 pad 13: HSPI_CLK -> Net-(U2-Pad13)
- U2 pad 14: HSPI_MISO -> Net-(U2-Pad14)
- U2 pad 16: HSPI_MOSI -> Net-(U2-Pad16)
- U2 pad 17: (no net) -> Net-(U2-Pad17)
- U2 pad 18: (no net) -> Net-(U2-Pad18)
- U2 pad 19: (no net) -> Net-(U2-Pad19)
- U2 pad 20: (no net) -> Net-(U2-Pad20)
- U2 pad 21: (no net) -> Net-(U2-Pad21)
- U2 pad 22: (no net) -> Net-(U2-Pad22)
- U2 pad 23: (no net) -> Net-(U2-Pad23)
- U2 pad 24: IO2 -> Net-(U2-Pad24)
- U2 pad 25: IO0 -> Net-(U2-Pad25)
- U2 pad 26: CAN_RX -> Net-(U2-Pad26)
- U2 pad 29: CAN_TX -> Net-(U2-Pad29)
- U2 pad 3: EN -> Net-(U2-Pad3)
- U2 pad 30: (no net) -> Net-(U2-Pad30)
- U2 pad 31: I2C_S_D -> Net-(U2-Pad31)
- U2 pad 33: I2C_S_C -> Net-(U2-Pad33)
- U2 pad 34: RX0 -> Net-(U2-Pad34)
- U2 pad 35: TX0 -> Net-(U2-Pad35)
- U2 pad 36: I2C_F_D -> Net-(U2-Pad36)
- U2 pad 37: I2C_F_C -> Net-(U2-Pad37)
- U2 pad 4: AN0 -> Net-(U2-Pad4)
- U2 pad 5: AN3 -> Net-(U2-Pad5)
- U2 pad 6: AN6 -> Net-(U2-Pad6)
- U2 pad 7: AN7 -> Net-(U2-Pad7)
- U2 pad 8: AN4 -> Net-(U2-Pad8)
- U2 pad 9: AN5 -> Net-(U2-Pad9)
Routing:
- net +3V3: track 200.5 -> 0.01 mm, vias 16 -> 0
- net +5V: track 120.6 -> 0.00 mm, vias 10 -> 0
- net EN: track 78.2 -> 0.00 mm, vias 2 -> 0
- net IO0: track 66.1 -> 0.00 mm, vias 2 -> 0
- net +12V: track 59.2 -> 0.00 mm, vias 5 -> 0
- net RX0: track 46.0 -> 0.00 mm
- net TX0: track 45.1 -> 0.00 mm
- net CAN_L: track 40.1 -> 0.00 mm, vias 2 -> 0
- net CAN_H: track 38.5 -> 0.00 mm, vias 2 -> 0
- net CAN_RX: track 37.1 -> 0.00 mm, vias 1 -> 0
- net IO2: track 35.9 -> 0.00 mm, vias 1 -> 0
- net CAN_TX: track 34.1 -> 0.00 mm, vias 1 -> 0
- net AN5: track 33.9 -> 0.00 mm, vias 2 -> 0
- net I2C_S_D: track 29.0 -> 0.00 mm, vias 1 -> 0
- net I2C_S_C: track 29.0 -> 0.00 mm, vias 1 -> 0
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- removed copper zone on B.Cu, net GND
- removed copper zone on F.Cu, net GND
Other:
- board size 40.9 x 63.5 mm -> 40.9 x 60 mm
- board text removed: "0"
- board text removed: "12"
- board text removed: "13"
- board text removed: "14"
- board text removed: "19"
- board text removed: "2"
- board text removed: "21"
- board text removed: "22"
- board text removed: "23"
- board text removed: "25"
- board text removed: "26"
- board text removed: "27"
- board text removed: "32"
- board text removed: "33"
- board text removed: "34"
- board text removed: "35"
- board text removed: "36"
- board text removed: "39"
- board text removed: "4"
- board text removed: "5"
- board text removed: "Hi"
