File: esp_wrover_open.sch (KiCad schematic (older format))
At the start: 44 parts, among them J1 USB_B_Micro, J2 Conn_02x13_Counter_Clockwise, J3 Barrel_Jack_Switch, J4 CAN_out, J5 Conn_02x03_Counter_Clockwise, J6 Conn_02x03_Counter_Clockwise, J7 Conn_02x03_Counter_Clockwise, J8 USB_C_Receptacle_USB2.0, Q3 Q_NPN_BCE, Q4 Q_NPN_BCE, SW1 reset, SW2 boot, U1 ESP32-WROVER-B_(16MB), U2 CP2102N, U3 AMS1117-3.3, U4 SN65HVD230, U5 LM1084-5.0

Commit message: update
Other:
- note added: "Header"
- note added: "USB_CAN"
- note added: "power 12V"
- moved on the sheet: J2, J8
Changed lines of the file:
@@
 	1    0    0    -1
 $EndComp
-Text GLabel 6600 4000 0    50   Input ~ 0
+Text GLabel 7200 3750 0    50   Input ~ 0
 AN0
 $Comp
 L Connector_Generic:Conn_02x13_Counter_Clockwise J2
 U 1 1 5F00C228
-P 6800 4600
-F 0 "J2" H 6850 5417 50  0000 C CNN
-F 1 "Conn_02x13_Counter_Clockwise" H 6850 5326 50  0000 C CNN
-F 2 "Connector_PinHeader_2.54mm:PinHeader_2x13_P2.54mm_Vertical" H 6800 4600 50  0001 C CNN
-F 3 "~" H 6800 4600 50  0001 C CNN
-	1    6800 4600
-	1    0    0    -1
-$EndComp
-Text GLabel 6600 4200 0    50   Input ~ 0
+P 7400 4350
+F 0 "J2" H 7450 5167 50  0000 C CNN
+F 1 "Conn_02x13_Counter_Clockwise" H 7450 5076 50  0000 C CNN
+F 2 "Connector_PinHeader_2.54mm:PinHeader_2x13_P2.54mm_Vertical" H 7400 4350 50  0001 C CNN
+F 3 "~" H 7400 4350 50  0001 C CNN
+	1    7400 4350
+	1    0    0    -1
+$EndComp
+Text GLabel 7200 3950 0    50   Input ~ 0
 AN3
-Text GLabel 6600 4400 0    50   Input ~ 0
+Text GLabel 7200 4150 0    50   Input ~ 0
 AN6
-Text GLabel 6600 4600 0    50   Input ~ 0
+Text GLabel 7200 4350 0    50   Input ~ 0
 AN7
-Text GLabel 6600 4800 0    50   Input ~ 0
+Text GLabel 7200 4550 0    50   Input ~ 0
 AN4
-Text GLabel 6600 5000 0    50   Input ~ 0
+Text GLabel 7200 4750 0    50   Input ~ 0
 DAC1
-Text GLabel 6600 5200 0    50   Input ~ 0
+Text GLabel 7200 4950 0    50   Input ~ 0
 DAC2
-Text GLabel 7100 4700 2    50   Input ~ 0
+Text GLabel 7700 4450 2    50   Input ~ 0
 HSPI_SE
-Text GLabel 7100 4500 2    50   Input ~ 0
+Text GLabel 7700 4250 2    50   Input ~ 0
 HSPI_CLK
-Text GLabel 7100 4300 2    50   Input ~ 0
+Text GLabel 7700 4050 2    50   Input ~ 0
 HSPI_MISO
-Text GLabel 7100 4100 2    50   Input ~ 0
+Text GLabel 7700 3850 2    50   Input ~ 0
 HSPI_MOSI
-Text GLabel 6600 4100 0    50   Input ~ 0
+Text GLabel 7200 3850 0    50   Input ~ 0
 I2C_F_C
-Text GLabel 6600 4300 0    50   Input ~ 0
+Text GLabel 7200 4050 0    50   Input ~ 0
 I2C_F_D
 $Comp
 L power:+3V3 #PWR0114
 U 1 1 5F039EA4
-P 7100 5100
-F 0 "#PWR0114" H 7100 4950 50  0001 C CNN
-F 1 "+3V3" V 7115 5228 50  0000 L CNN
-F 2 "" H 7100 5100 50  0001 C CNN
-F 3 "" H 7100 5100 50  0001 C CNN
-	1    7100 5100
+P 7700 4850
+F 0 "#PWR0114" H 7700 4700 50  0001 C CNN
+F 1 "+3V3" V 7715 4978 50  0000 L CNN
+F 2 "" H 7700 4850 50  0001 C CNN
+F 3 "" H 7700 4850 50  0001 C CNN
+	1    7700 4850
 	0    1    1    0
 $EndComp
@@
 L power:GND #PWR0115
 U 1 1 5F0397EB
-P 7100 4900
-F 0 "#PWR0115" H 7100 4650 50  0001 C CNN
-F 1 "GND" V 7105 4772 50  0000 R CNN
-F 2 "" H 7100 4900 50  0001 C CNN
-F 3 "" H 7100 4900 50  0001 C CNN
-	1    7100 4900
+P 7700 4650
+F 0 "#PWR0115" H 7700 4400 50  0001 C CNN
+F 1 "GND" V 7705 4522 50  0000 R CNN
+F 2 "" H 7700 4650 50  0001 C CNN
+F 3 "" H 7700 4650 50  0001 C CNN
+	1    7700 4650
 	0    -1   -1   0
 $EndComp
@@
 L power:+3V3 #PWR0116
 U 1 1 5F0462B8
-P 6600 4700
-F 0 "#PWR0116" H 6600 4550 50  0001 C CNN
-F 1 "+3V3" V 6615 4828 50  0000 L CNN
-F 2 "" H 6600 4700 50  0001 C CNN
-F 3 "" H 6600 4700 50  0001 C CNN
-	1    6600 4700
+P 7200 4450
+F 0 "#PWR0116" H 7200 4300 50  0001 C CNN
+F 1 "+3V3" V 7215 4578 50  0000 L CNN
+F 2 "" H 7200 4450 50  0001 C CNN
+F 3 "" H 7200 4450 50  0001 C CNN
+	1    7200 4450
 	0    -1   -1   0
 $EndComp
@@
 L power:GND #PWR0117
 U 1 1 5F04926E
-P 6600 4500
-F 0 "#PWR0117" H 6600 4250 50  0001 C CNN
-F 1 "GND" V 6605 4372 50  0000 R CNN
-F 2 "" H 6600 4500 50  0001 C CNN
-F 3 "" H 6600 4500 50  0001 C CNN
-	1    6600 4500
-	0    1    1    0
-$EndComp
-Text GLabel 6600 4900 0    50   Input ~ 0
+P 7200 4250
+F 0 "#PWR0117" H 7200 4000 50  0001 C CNN
+F 1 "GND" V 7205 4122 50  0000 R CNN
+F 2 "" H 7200 4250 50  0001 C CNN
+F 3 "" H 7200 4250 50  0001 C CNN
+	1    7200 4250
+	0    1    1    0
+$EndComp
+Text GLabel 7200 4650 0    50   Input ~ 0
 I2C_S_C
-Text GLabel 6600 5100 0    50   Input ~ 0
+Text GLabel 7200 4850 0    50   Input ~ 0
 I2C_S_D
 $Comp
 L power:+3V3 #PWR0118
 U 1 1 5F05020F
-P 7100 5000
-F 0 "#PWR0118" H 7100 4850 50  0001 C CNN
-F 1 "+3V3" V 7115 5128 50  0000 L CNN
-F 2 "" H 7100 5000 50  0001 C CNN
-F 3 "" H 7100 5000 50  0001 C CNN
-	1    7100 5000
+P 7700 4750
+F 0 "#PWR0118" H 7700 4600 50  0001 C CNN
+F 1 "+3V3" V 7715 4878 50  0000 L CNN
+F 2 "" H 7700 4750 50  0001 C CNN
+F 3 "" H 7700 4750 50  0001 C CNN
+	1    7700 4750
 	0    1    1    0
 $EndComp
@@
 L power:GND #PWR0119
 U 1 1 5F050215
-P 7100 5200
-F 0 "#PWR0119" H 7100 4950 50  0001 C CNN
-F 1 "GND" V 7105 5072 50  0000 R CNN
-F 2 "" H 7100 5200 50  0001 C CNN
-F 3 "" H 7100 5200 50  0001 C CNN
-	1    7100 5200
-	0    -1   -1   0
-$EndComp
-Text GLabel 7100 4800 2    50   Input ~ 0
+P 7700 4950
+F 0 "#PWR0119" H 7700 4700 50  0001 C CNN
+F 1 "GND" V 7705 4822 50  0000 R CNN
+F 2 "" H 7700 4950 50  0001 C CNN
+F 3 "" H 7700 4950 50  0001 C CNN
+	1    7700 4950
+	0    -1   -1   0
+$EndComp
+Text GLabel 7700 4550 2    50   Input ~ 0
 CAN_TX
-Text GLabel 7100 4600 2    50   Input ~ 0
+Text GLabel 7700 4350 2    50   Input ~ 0
 CAN_RX
-Text GLabel 7100 4400 2    50   Input ~ 0
+Text GLabel 7700 4150 2    50   Input ~ 0
 IO0
-Text GLabel 7100 4200 2    50   Input ~ 0
+Text GLabel 7700 3950 2    50   Input ~ 0
 IO2
 $Comp
@@
 L Connector:USB_C_Receptacle_USB2.0 J8
 U 1 1 5EF61382
-P 8750 4600
-F 0 "J8" H 8857 5467 50  0000 C CNN
-F 1 "USB_C_Receptacle_USB2.0" H 8857 5376 50  0000 C CNN
-F 2 "Connector_USB:USB_C_Receptacle_HRO_TYPE-C-31-M-12" H 8900 4600 50  0001 C CNN
-F 3 "https://www.usb.org/sites/default/files/documents/usb_type-c.zip" H 8900 4600 50  0001 C CNN
-	1    8750 4600
-	1    0    0    -1
-$EndComp
-Wire Wire Line
-	9350 4500 9350 4600
-Wire Wire Line
-	9350 4700 9350 4800
-Wire Wire Line
-	8450 5500 8600 5500
+P 9600 4350
+F 0 "J8" H 9707 5217 50  0000 C CNN
+F 1 "USB_C_Receptacle_USB2.0" H 9707 5126 50  0000 C CNN
+F 2 "Connector_USB:USB_C_Receptacle_HRO_TYPE-C-31-M-12" H 9750 4350 50  0001 C CNN
+F 3 "https://www.usb.org/sites/default/files/documents/usb_type-c.zip" H 9750 4350 50  0001 C CNN
+	1    9600 4350
+	1    0    0    -1
+$EndComp
+Wire Wire Line
+	10200 4250 10200 4350
+Wire Wire Line
+	10200 4450 10200 4550
+Wire Wire Line
+	9300 5250 9450 5250
 $Comp
 L power:GND #PWR0127
 U 1 1 5EF6C465
-P 8600 5500
-F 0 "#PWR0127" H 8600 5250 50  0001 C CNN
-F 1 "GND" H 8605 5327 50  0000 C CNN
-F 2 "" H 8600 5500 50  0001 C CNN
-F 3 "" H 8600 5500 50  0001 C CNN
-	1    8600 5500
-	1    0    0    -1
-$EndComp
-Connection ~ 8600 5500
-Wire Wire Line
-	8600 5500 8750 5500
+P 9450 5250
+F 0 "#PWR0127" H 9450 5000 50  0001 C CNN
+F 1 "GND" H 9455 5077 50  0000 C CNN
+F 2 "" H 9450 5250 50  0001 C CNN
+F 3 "" H 9450 5250 50  0001 C CNN
+	1    9450 5250
+	1    0    0    -1
+$EndComp
+Connection ~ 9450 5250
+Wire Wire Line
+	9450 5250 9600 5250
 $Comp
 L power:+12V #PWR0131
 U 1 1 5EF6FE81
-P 9350 4000
-F 0 "#PWR0131" H 9350 3850 50  0001 C CNN
-F 1 "+12V" H 9365 4173 50  0000 C CNN
-F 2 "" H 9350 4000 50  0001 C CNN
-F 3 "" H 9350 4000 50  0001 C CNN
-	1    9350 4000
-	1    0    0    -1
-$EndComp
-Text GLabel 9350 4750 2    50   Input ~ 0
+P 10200 3750
+F 0 "#PWR0131" H 10200 3600 50  0001 C CNN
+F 1 "+12V" H 10215 3923 50  0000 C CNN
+F 2 "" H 10200 3750 50  0001 C CNN
+F 3 "" H 10200 3750 50  0001 C CNN
+	1    10200 3750
+	1    0    0    -1
+$EndComp
+Text GLabel 10200 4500 2    50   Input ~ 0
 CAN_H
-Text GLabel 9350 4550 2    50   Input ~ 0
+Text GLabel 10200 4300 2    50   Input ~ 0
 CAN_L
-NoConn ~ 9350 4200
-NoConn ~ 9350 4300
-NoConn ~ 9350 5100
-NoConn ~ 9350 5200
+NoConn ~ 10200 3950
+NoConn ~ 10200 4050
+NoConn ~ 10200 4850
+NoConn ~ 10200 4950
 $Comp
 L Regulator_Linear:LM1084-5.0 U5
@@
 	0    -1   -1   0
 $EndComp
-Text GLabel 7100 4000 2    50   Input ~ 0
+Text GLabel 7700 3750 2    50   Input ~ 0
 AN5
+Wire Notes Line
+	6050 3600 8400 3600
+Wire Notes Line
+	8400 3600 8400 5000
+Wire Notes Line
+	8400 5000 6050 5000
+Wire Notes Line
+	6050 5000 6050 3600
+Wire Notes Line
+	8850 3600 10750 3600
+Wire Notes Line
+	10750 3600 10750 5500
+Wire Notes Line
+	10750 5500 8850 5500
+Wire Notes Line
+	8850 5500 8850 3600
+Wire Notes Line
+	4350 5050 6850 5050
+Wire Notes Line
+	6850 5050 6850 7700
+Wire Notes Line
+	6850 7700 4350 7700
+Wire Notes Line
+	4350 7700 4350 5050
+Text Notes 4450 5200 0    79   ~ 16
+power 12V
+Text Notes 6150 4900 0    79   ~ 16
+Header
+Text Notes 10100 5400 0    79   ~ 16
+USB_CAN
 $EndSCHEMATC

Commit message: cpmonent
Parts:
- removed C10, C8: 10uF, Resistor_SMD:R_1210_3225Metric, symbol Device:C
- removed C11, C9: 100nF, Capacitor_SMD:C_0603_1608Metric, symbol Device:C
- removed J1: USB_B_Micro, Connector_USB:USB_Micro-B_Wuerth_629105150521, symbol Connector:USB_B_Micro
- removed J2: Conn_02x13_Counter_Clockwise, Connector_PinHeader_2.54mm:PinHeader_2x13_P2.54mm_Vertical, symbol Connector_Generic:Conn_02x13_Counter_Clockwise
- removed J4: CAN_out, Connector:JWT_A3963_1x02_P3.96mm_Vertical, symbol Connector_Generic:Conn_01x02
- removed J5: Conn_02x03_Counter_Clockwise, Connector_PinHeader_2.54mm:PinHeader_2x03_P2.54mm_Vertical, symbol Connector_Generic:Conn_02x03_Counter_Clockwise
- removed R14: 1K, Resistor_SMD:R_0603_1608Metric_Pad1.05x0.95mm_HandSolder, symbol Device:R
- removed R3: 10K, Resistor_SMD:R_0603_1608Metric_Pad1.05x0.95mm_HandSolder, symbol Device:R
- removed R4: 120, Resistor_SMD:R_0603_1608Metric_Pad1.05x0.95mm_HandSolder, symbol Device:R
- removed U2: CP2102N, Package_DFN_QFN:QFN-28-1EP_5x5mm_P0.5mm_EP3.35x3.35mm, symbol Interface_USB:CP2102N-A01-GQFN28
- removed U4: SN65HVD230, Package_SO:SOIC-8_3.9x4.9mm_P1.27mm, symbol Interface_CAN_LIN:SN65HVD230
- removed U5: LM1084-5.0, Package_TO_SOT_THT:TO-220-3_Vertical, symbol Regulator_Linear:LM1084-5.0
- added J5: Conn_02x20_Counter_Clockwise, Connector_PinHeader_2.54mm:PinHeader_2x20_P2.54mm_Vertical, symbol Connector_Generic:Conn_02x20_Counter_Clockwise
- added U1: CP2104, Package_DFN_QFN:QFN-24-1EP_4x4mm_P0.5mm_EP2.6x2.6mm, symbol Interface_USB:CP2104
- J1: renamed from J8; symbol Connector:USB_C_Receptacle_USB2.0 -> esp_wrover_open-rescue:USB_C_Receptacle_USB2.0-Connector
- renumbered D3 to D1, D4 to D2, D5 to D3, J3 to J2, J6 to J3, J7 to J4, Q3 to Q1, Q4 to Q2, R16 to R10, R9 to R3, R10 to R4, R13 to R5, R15 to R6, R11 to R7, R12 to R8, R17 to R9, U1 to U2
Connections:
- net +12V is gone; now on net +5V: J1.A4 (VBUS), J1.A9 (VBUS), J1.B4 (VBUS), J1.B9 (VBUS)
- net +3V3: now also J5.13 (Pin_13), J5.39 (Pin_39), J5.5 (Pin_5)
- net +5V: now also J5.4 (Pin_4), J5.40 (Pin_40), U1.7 (REGIN), U1.8 (VBUS)
- net DTR: now also U1.23 (DTR)
- net EN: now also J5.1 (Pin_1); no longer U2.3 (EN)
- net GND: now also J5.14 (Pin_14), J5.37 (Pin_37), J5.38 (Pin_38), J5.6 (Pin_6), U1.2 (GND), U1.25 (PAD)
- net IO0: no longer U2.25 (IO0/GPIO0/ADC2_CH1/TOUCH1/RTC_GPIO11/CLK_OUT1/EMAC_TX_CLK)
- net RTS: now also U1.19 (RTS)
- net RX0: now also R7.1, J5.2 (Pin_2); no longer R8.1, U2.34 (RXD0/GPIO3/U0RXD/CLK_OUT2)
- net SU-: now also U1.15 (~SUSPEND)
- net TX0: now also R8.1, J5.3 (Pin_3); no longer R7.1, U2.35 (TXD0/GPIO1/U0TXD/CLK_OUT3/EMAC_RXD2)
- net at R7.2: now also U1.21 (TXD)
- net at R8.2: now also U1.20 (RXD)
- net AN0: no longer names the net of U2.4 (SENSOR_VP/GPIO36/ADC1_CH0/RTC_GPIO0)
- net AN3: no longer names the net of U2.5 (SENSOR_VN/GPIO39/ADC1_CH3/RTC_GPIO3)
- net AN4: no longer names the net of U2.8 (IO32/GPIO32/XTAL_32K_P/ADC1_CH4/TOUCH9/RTC_GPIO9)
- net AN5: no longer names the net of U2.9 (IO33/GPIO33/XTAL_32K_N/ADC1_CH5/TOUCH8/RTC_GPIO8)
- net AN6: no longer names the net of U2.6 (IO34/GPIO34/ADC1_CH6/RTC_GPIO4)
- net AN7: no longer names the net of U2.7 (IO35/GPIO35/ADC1_CH7/RTC_GPIO5)
- net CAN_H: no longer names the net of J1.A6 (D+), J1.B6 (D+)
- net CAN_H: now also U1.3 (D+)
- net CAN_L: no longer names the net of J1.A7 (D-), J1.B7 (D-)
- net CAN_L: now also U1.4 (D-)
- net CAN_RX: no longer names the net of U2.26 (IO4/GPIO4/ADC2_CH0/TOUCH0/RTC_GPIO10/HSPIHD/HS2_DATA1/SD_DATA1/EMAC_TX_ER)
- net CAN_TX: no longer names the net of U2.29 (IO5/GPIO5/VSPICS0/HS1_DATA6/EMAC_RX_CLK)
- net DAC1: no longer names the net of U2.10 (IO25/GPIO25/DAC_1/ADC2_CH8/RTC_GPIO6/EMAC_RXD0)
- net DAC2: no longer names the net of U2.11 (IO26/DAC_2/ADC2_CH9/RTC_GPIO7/EMAC_RXD1)
- net HSPI_CLK: no longer names the net of U2.13 (IO14/GPIO14/ADC2_CH6/TOUCH6/RTC_GPIO16/MTMS/HSPICLK/HS2_CLK/SD_CLK/EMAC_TXD2)
- net HSPI_MISO: no longer names the net of U2.14 (IO12/GPIO12/ADC2_CH5/TOUCH5/RTC_GPIO15/HSPIQ/HS2_DATA2/SD_DATA2/EMAC_TXD3)
- net HSPI_MOSI: no longer names the net of U2.16 (IO13/GPIO13/ADC2_CH4/TOUCH4/RTC_GPIO14/MTCK/HSPID/HS2_DATA3/SD_DATA3/EMAC_RX_ER)
- net HSPI_SE: no longer names the net of U2.12 (IO27/GPIO27/ADC2_CH7/TOUCH7/RTC_GPIO17/EMAC_RX_DV)
- net I2C_F_C: no longer names the net of U2.37 (IO23/GPIO23/VSPID/HS1_STROBE)
- net I2C_F_D: no longer names the net of U2.36 (IO22/GPIO22/VSPIWP/U0RTS/EMAC_TXD1)
- net I2C_S_C: no longer names the net of U2.33 (IO21/GPIO21/VSPIHD/EMAC_TX_EN)
- net I2C_S_D: no longer names the net of U2.31 (IO19/GPIO19/VSPIQ/U0CTS/EMAC_TXD0)
- net IO15: no longer names the net of U2.23 (IO15/GPIO15/ADC2_CH3/TOUCH3/MTDO/HSPICS0/RTC_GPIO13/HS2_CMD/SD_CMD/EMAC_RXD3)
- net IO18: no longer names the net of U2.30 (IO18/GPIO18/VSPICLK/HS1_DATA7)
- net IO2: no longer names the net of U2.24 (IO2/GPIO2/ADC2_CH2/TOUCH2/RTC_GPIO12/HSPIWP/HS2_DATA0/SD_DATA0)
- new net 0: J5.15 (Pin_15)
- new net 12: J5.19 (Pin_19)
- new net 13: J5.20 (Pin_20)
- new net 14: J5.21 (Pin_21)
- new net 15: J5.22 (Pin_22)
- new net 18: J5.23 (Pin_23)
- new net 19: J5.24 (Pin_24)
- new net 2: J5.16 (Pin_16)
- new net 21: J5.25 (Pin_25)
- new net 22: J5.26 (Pin_26)
- new net 23: J5.27 (Pin_27)
- new net 25: J5.28 (Pin_28)
- new net 26: J5.29 (Pin_29)
- new net 27: J5.30 (Pin_30)
- new net 32: J5.31 (Pin_31)
- new net 33: J5.32 (Pin_32)
- new net 34: J5.33 (Pin_33)
- new net 35: J5.34 (Pin_34)
- new net 36: J5.35 (Pin_35)
- new net 39: J5.36 (Pin_36)
- new net 4: J5.17 (Pin_17)
- new net 5: J5.18 (Pin_18)
- new net CMD: J5.12 (Pin_12)
- new net SCK: J5.7 (Pin_7)
- new net SD0: J5.8 (Pin_8)
- new net SD1: J5.9 (Pin_9)
- new net SD2: J5.10 (Pin_10)
- new net SD3: J5.11 (Pin_11)
- no-connect marks 26 -> 18
Other:
- note removed: "CAN"
- note removed: "Power\n"
- note removed: "USB_CAN"
- note removed: "power 12V"
- moved on the sheet: C3, C4, C5, D1, D2, D3, J1, J2, J3, J4, Q1, Q2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
